File: KiCad/4bitDAC.sch (KiCad schematic (older format))
At the start: 12 parts, among them P1 CONN_01X04, P2 CONN_01X04, U1 LM741

Commit message: In process of editing PCB.
Parts:
- P1: renamed from P2; footprint Pin_Headers:Pin_Header_Straight_1x04 -> Pin_Headers:Pin_Header_Straight_1x04_Pitch2.54mm
- P2: renamed from P1; footprint Pin_Headers:Pin_Header_Straight_1x04 -> Pin_Headers:Pin_Header_Straight_1x04_Pitch2.54mm
- R1: renamed from R7; footprint Resistors_SMD:R_0805_HandSoldering -> Resistors_Universal:Resistor_SMD+THTuniversal_0805to1206_RM10_HandSoldering
- R2: renamed from R8; footprint Resistors_SMD:R_0805_HandSoldering -> Resistors_Universal:Resistor_SMD+THTuniversal_0805to1206_RM10_HandSoldering
- R3: renamed from R2; footprint Resistors_SMD:R_0805_HandSoldering -> Resistors_Universal:Resistor_SMD+THTuniversal_0805to1206_RM10_HandSoldering
- R4: renamed from R3; footprint Resistors_SMD:R_0805_HandSoldering -> Resistors_Universal:Resistor_SMD+THTuniversal_0805to1206_RM10_HandSoldering
- R5: renamed from R4; footprint Resistors_SMD:R_0805_HandSoldering -> Resistors_Universal:Resistor_SMD+THTuniversal_0805to1206_RM10_HandSoldering
- R6: renamed from R5; footprint Resistors_SMD:R_0805_HandSoldering -> Resistors_Universal:Resistor_SMD+THTuniversal_0805to1206_RM10_HandSoldering
- R7: renamed from R1; footprint Resistors_SMD:R_0805_HandSoldering -> Resistors_Universal:Resistor_SMD+THTuniversal_0805to1206_RM10_HandSoldering
- R8: renamed from R6; footprint Resistors_SMD:R_0805_HandSoldering -> Resistors_Universal:Resistor_SMD+THTuniversal_0805to1206_RM10_HandSoldering
- RV1: footprint (none) -> Potentiometers:Potentiometer_Trimmer_ACP_CA9h2.5_Vertical_Px2.5mm_Py5.0mm
- U1: footprint Housings_DIP:DIP-8_W7.62mm -> Housings_DIP:DIP-8_W7.62mm_LongPads
Connections:
- net D3: now reaches P2.4 (P4), R3.2, R4.2
- net D1: now reaches P2.2 (P2), R6.2
- net D0: now reaches P2.1 (P1), R7.2
- net D2: now reaches P2.3 (P3), R5.2
Other:
- moved on the sheet: P1, P2, R1, R2, R3, R4, R5, R6, R7, R8, RV1, U1
